Commit message: Start MoveIt on request, fix localization stamps, reduce load, harden stop_sim
- bringup.launch.py: moveit defaults to False; start MoveIt with moveit:=True.
  Launch arguments renamed to teleop, gazebo_gui, gazebo_gui_delay.
- neo_localization2: compute the pose expiry stamp with rclcpp time
  arithmetic instead of adding 1e9 to nanosec.
- Odometry published at 50 Hz (control loop stays at 100 Hz), controller
  state topics at 50 Hz, RViz frame rate 10 instead of 30.
- navigation.yaml: use_sim_time for all nodes.
- stop_sim.sh: stop the whole process tree of every launch, then orphans,
  escalating SIGINT, SIGTERM, SIGKILL.
- package.xml: declare RViz plugins, xterm and neo_sim_objects.

File: neo_simulation2/components/common_macro/gazebo_object_controller_macro.xacro (robot description, xacro)
@@ -22,6 +22,4 @@
                 <robotNamespace><remapping>/tf:=tf</remapping></robotNamespace>
                 <ros>    <remapping>/tf:=tf</remapping>    </ros>
-                <!-- Set odom publish rate -->
-                <odometryRate>${odom_update_rate}</odometryRate>
                 <!-- Control loop rate, i.e. how often the commanded velocity is
                      re-applied (the real omnidrive runs at control_rate 100 Hz).
@@ -30,6 +28,8 @@
                      of the commanded speed. -->
                 <update_rate>${controller_update_rate}</update_rate>
-                <!-- Odometry and odom TF publish rate -->
-                <publish_rate>${controller_update_rate}</publish_rate>
+                <!-- Odometry and odom TF publish rate. Independent of the control
+                     loop, so it can be lowered without slowing the base. (The
+                     plugin has no odometryRate parameter; this is the one it reads.) -->
+                <publish_rate>${odom_update_rate}</publish_rate>
                 <!-- Stop when cmd_vel goes quiet for this long (s). 0 disables. -->
                 <cmd_timeout>${cmd_timeout}</cmd_timeout>

File: neo_simulation2/robots/mpo_700/urdf/mpo_700_gazebo.urdf.xacro (robot description, xacro)
@@ -19,6 +19,11 @@
     <xacro:property name="lidar_1_update_rate" value="20" />
     <xacro:property name="lidar_2_update_rate" value="20" />
+    <!-- Base control loop stays at 100 Hz: the commanded velocity must be
+         re-applied often enough that wheel friction cannot slow the base between
+         updates. Odometry (odom topic and odom TF) is published at 50 Hz to
+         reduce message load; Nav2's controller runs at 50 Hz, so it still gets
+         one odometry update per control cycle. -->
     <xacro:property name="controller_update_rate" value="100" />
-    <xacro:property name="odom_update_rate" value="100" />
+    <xacro:property name="odom_update_rate" value="50" />
     <!--Object Controller-->
     <xacro:gazebo_object_controller
