Commit message: Add pick-and-place arm poses and 90 % gripper poses to MoveIt
- ur_manipulator named states for the mission stages (home, pre_grasp,
  grasp, lift, pre_place, place, retreat), values from Stage_values.md.
- gripper named states: open 0.07, close 0.63 (90 % of the 0.0-0.7 range).

File: neo_mpo_moveit2/neo_ur_moveit_config/srdf/mpo_700.srdf.xacro (robot description, xacro)
@@ -39,4 +39,25 @@
       <joint name="${prefix_value}wrist_3_joint" value="-0.11" />
     </group_state>
+    <!-- Stages of the pick-and-place mission (Stage_values.md). Joint values in the
+         order shoulder_pan, shoulder_lift, elbow, wrist_1, wrist_2, wrist_3 (rad).
+         All poses except home are valid only with the robot at the recorded pick and
+         place positions. -->
+    <xacro:macro name="stage_pose" params="name pan lift elbow w1 w2 w3">
+      <group_state name="${name}" group="ur_manipulator">
+        <joint name="${prefix_value}shoulder_pan_joint" value="${pan}" />
+        <joint name="${prefix_value}shoulder_lift_joint" value="${lift}" />
+        <joint name="${prefix_value}elbow_joint" value="${elbow}" />
+        <joint name="${prefix_value}wrist_1_joint" value="${w1}" />
+        <joint name="${prefix_value}wrist_2_joint" value="${w2}" />
+        <joint name="${prefix_value}wrist_3_joint" value="${w3}" />
+      </group_state>
+    </xacro:macro>
+    <xacro:stage_pose name="home"      pan="1.49" lift="-2.50" elbow="2.00" w1="0.00"  w2="-1.49" w3="0.01"/>
+    <xacro:stage_pose name="pre_grasp" pan="1.23" lift="-1.97" elbow="2.27" w1="-1.89" w2="-1.57" w3="-1.90"/>
+    <xacro:stage_pose name="grasp"     pan="1.23" lift="-1.79" elbow="2.48" w1="-2.25" w2="-1.57" w3="-1.91"/>
+    <xacro:stage_pose name="lift"      pan="1.23" lift="-1.92" elbow="2.35" w1="-2.00" w2="-1.57" w3="-1.91"/>
+    <xacro:stage_pose name="pre_place" pan="1.17" lift="-1.96" elbow="2.27" w1="-1.88" w2="-1.56" w3="-1.96"/>
+    <xacro:stage_pose name="place"     pan="1.18" lift="-1.80" elbow="2.47" w1="-2.24" w2="-1.57" w3="-1.97"/>
+    <xacro:stage_pose name="retreat"   pan="1.18" lift="-1.97" elbow="2.28" w1="-1.88" w2="-1.57" w3="-1.97"/>
     <!--DISABLE COLLISIONS: By default it is assumed that any link of the robot could potentially come into collision with any other link in the robot. This tag disables collision checking between a specified pair of links. -->
     <disable_collisions link1="base_footprint" link2="cabinet_link" reason="Adjacent"/>

File: neo_mpo_moveit2/neo_ur_moveit_config/srdf/robotiq_2f_140.xacro (robot description, xacro)
@@ -15,11 +15,17 @@
     <passive_joint name="left_inner_knuckle_joint"/>
     <passive_joint name="left_inner_finger_joint"/>
+    <!-- Inside the full range (0.0 to 0.7), so that the fingers do not collide:
+         open 0.07, close 0.63 (90 % open / 90 % closed) -->
     <group_state name="open" group="gripper">
-      <joint name="finger_joint" value="0.0" />
+      <joint name="finger_joint" value="0.07" />
     </group_state>
     <group_state name="close" group="gripper">
-      <joint name="finger_joint" value="0.7" />
+      <joint name="finger_joint" value="0.63" />
     </group_state>
     <end_effector name="endeffector" parent_link="${prefix_value}wrist_3_link" group="gripper"/>
+    <!-- No collision checking for the contact pads, neither with other robot links
+         nor with objects in the planning scene (cube, tables) -->
+    <disable_default_collisions link="left_inner_finger_pad"/>
+    <disable_default_collisions link="right_inner_finger_pad"/>
     <disable_collisions link1="left_inner_finger" link2="ur_to_robotiq_link" reason="Never"/>
     <disable_collisions link1="left_inner_finger_pad" link2="ur_to_robotiq_link" reason="Never"/>

Commit message: Turn the gripper only 20 deg to the grasp poses; add grasp_cube
- wrist_3 of pre_grasp ... retreat turned by 90 deg (e.g. grasp -1.91 -> -0.34):
  the cube is square, so the fingers still line up with its faces, and the
  gripper turns about 20 deg from home instead of 110 deg. Grasp points unchanged.
- New gripper pose grasp_cube (finger_joint 0.265): closed around the 80 mm
  cube; measured in Gazebo, the fingers touch it at 0.267.

File: neo_mpo_moveit2/neo_ur_moveit_config/srdf/mpo_700.srdf.xacro (robot description, xacro)
@@ -42,5 +42,9 @@
          order shoulder_pan, shoulder_lift, elbow, wrist_1, wrist_2, wrist_3 (rad).
          All poses except home are valid only with the robot at the recorded pick and
-         place positions. -->
+         place positions.
+         wrist_3 is turned by 90 deg compared with the recorded values (e.g. grasp -1.91 ->
+         -0.34): the cube is square, so the fingers line up with its faces either way, and
+         the gripper then turns only about 20 deg from home instead of 110 deg. The grasp
+         point is unchanged; the fingers close sideways instead of front to back. -->
     <xacro:macro name="stage_pose" params="name pan lift elbow w1 w2 w3">
       <group_state name="${name}" group="ur_manipulator">
@@ -54,10 +58,10 @@
     </xacro:macro>
     <xacro:stage_pose name="home"      pan="1.49" lift="-2.50" elbow="2.00" w1="0.00"  w2="-1.49" w3="0.01"/>
-    <xacro:stage_pose name="pre_grasp" pan="1.23" lift="-1.97" elbow="2.27" w1="-1.89" w2="-1.57" w3="-1.90"/>
-    <xacro:stage_pose name="grasp"     pan="1.23" lift="-1.79" elbow="2.48" w1="-2.25" w2="-1.57" w3="-1.91"/>
-    <xacro:stage_pose name="lift"      pan="1.23" lift="-1.92" elbow="2.35" w1="-2.00" w2="-1.57" w3="-1.91"/>
-    <xacro:stage_pose name="pre_place" pan="1.17" lift="-1.96" elbow="2.27" w1="-1.88" w2="-1.56" w3="-1.96"/>
-    <xacro:stage_pose name="place"     pan="1.18" lift="-1.80" elbow="2.47" w1="-2.24" w2="-1.57" w3="-1.97"/>
-    <xacro:stage_pose name="retreat"   pan="1.18" lift="-1.97" elbow="2.28" w1="-1.88" w2="-1.57" w3="-1.97"/>
+    <xacro:stage_pose name="pre_grasp" pan="1.23" lift="-1.97" elbow="2.27" w1="-1.89" w2="-1.57" w3="-0.33"/>
+    <xacro:stage_pose name="grasp"     pan="1.23" lift="-1.79" elbow="2.48" w1="-2.25" w2="-1.57" w3="-0.34"/>
+    <xacro:stage_pose name="lift"      pan="1.23" lift="-1.92" elbow="2.35" w1="-2.00" w2="-1.57" w3="-0.34"/>
+    <xacro:stage_pose name="pre_place" pan="1.17" lift="-1.96" elbow="2.27" w1="-1.88" w2="-1.56" w3="-0.39"/>
+    <xacro:stage_pose name="place"     pan="1.18" lift="-1.80" elbow="2.47" w1="-2.24" w2="-1.57" w3="-0.40"/>
+    <xacro:stage_pose name="retreat"   pan="1.18" lift="-1.97" elbow="2.28" w1="-1.88" w2="-1.57" w3="-0.40"/>
     <!--DISABLE COLLISIONS: By default it is assumed that any link of the robot could potentially come into collision with any other link in the robot. This tag disables collision checking between a specified pair of links. -->
     <disable_collisions link1="base_footprint" link2="cabinet_link" reason="Adjacent"/>

File: neo_mpo_moveit2/neo_ur_moveit_config/srdf/robotiq_2f_140.xacro (robot description, xacro)
@@ -22,4 +22,11 @@
     <group_state name="close" group="gripper">
       <joint name="finger_joint" value="0.63" />
+    </group_state>
+    <!-- Closed around the 80 mm cube of neo_sim_objects/config/objects.yaml. Measured
+         in Gazebo: the fingers touch the centred cube at 0.267. Fingers and cube do not
+         collide (spawn_objects sets this), so closing further (close) would only make
+         the fingers pass into the cube. -->
+    <group_state name="grasp_cube" group="gripper">
+      <joint name="finger_joint" value="0.265" />
     </group_state>
     <end_effector name="endeffector" parent_link="${prefix_value}wrist_3_link" group="gripper"/>

Commit message: Separate platform and arm instructions; reduce the arm to three poses
- README section 1: overview of the parts that move separately (mobile
  platform, manipulator arm, gripper); each heading names its part. New
  section 1.5 moves the arm into the mission poses in RViz. Pick, place
  and home positions named as in Stage_values.md.
- MoveIt named states of the arm reduced to home, pregrasp and grasp;
  pregrasp and grasp are used at both tables, for picking and placing.
  lift, pre_place, retreat, place and test_configuration removed.
- Stage_values.md: shorter arm pose section, stages renumbered S0 to S10.

File: neo_mpo_moveit2/neo_ur_moveit_config/srdf/mpo_700.srdf.xacro (robot description, xacro)
@@ -31,16 +31,15 @@
       <joint name="${prefix_value}wrist_3_joint" value="0" />
     </group_state>
-    <group_state name="test_configuration" group="ur_manipulator">
-      <joint name="${prefix_value}elbow_joint" value="1.4" />
-      <joint name="${prefix_value}shoulder_lift_joint" value="-1.62" />
-      <joint name="${prefix_value}shoulder_pan_joint" value="1.54" />
-      <joint name="${prefix_value}wrist_1_joint" value="-1.2" />
-      <joint name="${prefix_value}wrist_2_joint" value="-1.6" />
-      <joint name="${prefix_value}wrist_3_joint" value="-0.11" />
-    </group_state>
-    <!-- Stages of the pick-and-place mission (Stage_values.md). Joint values in the
+    <!-- Arm poses of the pick-and-place mission (Stage_values.md). Joint values in the
          order shoulder_pan, shoulder_lift, elbow, wrist_1, wrist_2, wrist_3 (rad).
-         All poses except home are valid only with the robot at the recorded pick and
-         place positions.
+         Three poses cover the whole mission; pregrasp and grasp are used at the pick
+         table and at the place table:
+           home      travel pose, arm folded above the platform
+           pregrasp  gripper 16 cm above the grasp/place point: before grasping, lifting
+                     the cube, before placing, moving away after placing
+           grasp     gripper at the grasp/place point: grasping and placing the cube
+         The recorded lift, pre-place and retreat poses differed from pregrasp, and the
+         recorded place pose from grasp, by at most 0.11 rad per joint. pregrasp and
+         grasp are valid only with the robot at the pick or place position.
          wrist_3 is turned by 90 deg compared with the recorded values (e.g. grasp -1.91 ->
          -0.34): the cube is square, so the fingers line up with its faces either way, and
@@ -57,11 +56,7 @@
       </group_state>
     </xacro:macro>
-    <xacro:stage_pose name="home"      pan="1.49" lift="-2.50" elbow="2.00" w1="0.00"  w2="-1.49" w3="0.01"/>
-    <xacro:stage_pose name="pre_grasp" pan="1.23" lift="-1.97" elbow="2.27" w1="-1.89" w2="-1.57" w3="-0.33"/>
-    <xacro:stage_pose name="grasp"     pan="1.23" lift="-1.79" elbow="2.48" w1="-2.25" w2="-1.57" w3="-0.34"/>
-    <xacro:stage_pose name="lift"      pan="1.23" lift="-1.92" elbow="2.35" w1="-2.00" w2="-1.57" w3="-0.34"/>
-    <xacro:stage_pose name="pre_place" pan="1.17" lift="-1.96" elbow="2.27" w1="-1.88" w2="-1.56" w3="-0.39"/>
-    <xacro:stage_pose name="place"     pan="1.18" lift="-1.80" elbow="2.47" w1="-2.24" w2="-1.57" w3="-0.40"/>
-    <xacro:stage_pose name="retreat"   pan="1.18" lift="-1.97" elbow="2.28" w1="-1.88" w2="-1.57" w3="-0.40"/>
+    <xacro:stage_pose name="home"     pan="1.49" lift="-2.50" elbow="2.00" w1="0.00"  w2="-1.49" w3="0.01"/>
+    <xacro:stage_pose name="pregrasp" pan="1.23" lift="-1.97" elbow="2.27" w1="-1.89" w2="-1.57" w3="-0.33"/>
+    <xacro:stage_pose name="grasp"    pan="1.23" lift="-1.79" elbow="2.48" w1="-2.25" w2="-1.57" w3="-0.34"/>
     <!--DISABLE COLLISIONS: By default it is assumed that any link of the robot could potentially come into collision with any other link in the robot. This tag disables collision checking between a specified pair of links. -->
     <disable_collisions link1="base_footprint" link2="cabinet_link" reason="Adjacent"/>
